Commit message: 2025.4.27

File: src/robot_description/urdf/tiangong_lite.urdf (robot description, URDF)
Before this commit: robot tiangong_lite, 31 links, 30 joints
Links:
- link ankle_Pitch_l_link: geometry collision mesh filename=package://robot_description/meshes/ankle_Pitch_l_link.STL; visual mesh filename=package://robot_description/meshes/ankle_Pitch_l_link.STL
- link ankle_Pitch_r_link: geometry collision mesh filename=package://robot_description/meshes/ankle_Pitch_r_link.STL; visual mesh filename=package://robot_description/meshes/ankle_Pitch_r_link.STL
- link ankle_Roll_l_link: geometry collision mesh filename=package://robot_description/meshes/ankle_Roll_l_link.STL; visual mesh filename=package://robot_description/meshes/ankle_Roll_l_link.STL
- link ankle_Roll_r_link: geometry collision mesh filename=package://robot_description/meshes/ankle_Roll_r_link.STL; visual mesh filename=package://robot_description/meshes/ankle_Roll_r_link.STL
- link arm_fixed_l_link: geometry collision mesh filename=package://robot_description/meshes/arm_fixed_l_link.STL; visual mesh filename=package://robot_description/meshes/arm_fixed_l_link.STL
- link arm_fixed_r_link: geometry collision mesh filename=package://robot_description/meshes/arm_fixed_r_link.STL; visual mesh filename=package://robot_description/meshes/arm_fixed_r_link.STL
- link arm_yaw_l_link: geometry collision mesh filename=package://robot_description/meshes/arm_yaw_l_link.STL; visual mesh filename=package://robot_description/meshes/arm_yaw_l_link.STL
- link arm_yaw_r_link: geometry collision mesh filename=package://robot_description/meshes/arm_yaw_r_link.STL; visual mesh filename=package://robot_description/meshes/arm_yaw_r_link.STL
- link body_yaw_link: geometry collision mesh filename=package://robot_description/meshes/body_yaw_link.STL; visual mesh filename=package://robot_description/meshes/body_yaw_link.STL
- link elbow_pitch_l_link: geometry collision mesh filename=package://robot_description/meshes/elbow_pitch_l_link.STL; visual mesh filename=package://robot_description/meshes/elbow_pitch_l_link.STL
- link elbow_pitch_r_link: geometry collision mesh filename=package://robot_description/meshes/elbow_pitch_r_link.STL; visual mesh filename=package://robot_description/meshes/elbow_pitch_r_link.STL
- link head_fixed_link: geometry collision mesh filename=package://robot_description/meshes/head_fixed_link.STL; visual mesh filename=package://robot_description/meshes/head_fixed_link.STL
- link hip_Pitch_l_link: geometry collision mesh filename=package://robot_description/meshes/hip_Pitch_l_link.STL; visual mesh filename=package://robot_description/meshes/hip_Pitch_l_link.STL
- link hip_Pitch_r_link: geometry collision mesh filename=package://robot_description/meshes/hip_Pitch_r_link.STL; visual mesh filename=package://robot_description/meshes/hip_Pitch_r_link.STL
- link hip_Roll_l_link: geometry collision mesh filename=package://robot_description/meshes/hip_Roll_l_link.STL; visual mesh filename=package://robot_description/meshes/hip_Roll_l_link.STL
- link hip_Roll_r_link: geometry collision mesh filename=package://robot_description/meshes/hip_Roll_r_link.STL; visual mesh filename=package://robot_description/meshes/hip_Roll_r_link.STL
- link hip_Yaw_l_link: geometry collision mesh filename=package://robot_description/meshes/hip_Yaw_l_link.STL; visual mesh filename=package://robot_description/meshes/hip_Yaw_l_link.STL
- link hip_Yaw_r_link: geometry collision mesh filename=package://robot_description/meshes/hip_Yaw_r_link.STL; visual mesh filename=package://robot_description/meshes/hip_Yaw_r_link.STL
- link knee_Pitch_l_link: geometry collision mesh filename=package://robot_description/meshes/knee_Pitch_l_link.STL; visual mesh filename=package://robot_description/meshes/knee_Pitch_l_link.STL
- link knee_Pitch_r_link: geometry collision mesh filename=package://robot_description/meshes/knee_Pitch_r_link.STL; visual mesh filename=package://robot_description/meshes/knee_Pitch_r_link.STL
- link pelvis: geometry collision mesh filename=package://robot_description/meshes/pelvis.STL; visual mesh filename=package://robot_description/meshes/pelvis.STL
- link shoulder_pitch_l_link: geometry collision mesh filename=package://robot_description/meshes/shoulder_pitch_l_link.STL; visual mesh filename=package://robot_description/meshes/shoulder_pitch_l_link.STL
- link shoulder_pitch_r_link: geometry collision mesh filename=package://robot_description/meshes/shoulder_pitch_r_link.STL; visual mesh filename=package://robot_description/meshes/shoulder_pitch_r_link.STL
- link shoulder_roll_l_link: geometry collision mesh filename=package://robot_description/meshes/shoulder_roll_l_link.STL; visual mesh filename=package://robot_description/meshes/shoulder_roll_l_link.STL
- link shoulder_roll_r_link: geometry collision mesh filename=package://robot_description/meshes/shoulder_roll_r_link.STL; visual mesh filename=package://robot_description/meshes/shoulder_roll_r_link.STL
